File: stm32f103c8t6.kicad_pcb (KiCad board)
At the start: 2 copper layers, 28 parts, among them J1 USB_B_Micro, J2 Conn_01x04_Pin, J3 Conn_01x04_Pin, J4 Conn_01x04_Pin, SW1 SW_SPDT, U1 AMS1117-3.3, U2 STM32F103C8Tx, Y1 16Mhz

Commit message: Layouting don't compleate
Parts:
- moved C13 90.0 mm to (42.8, 85.7), turned to -135 degrees
- moved C9 89.0 mm to (46.0, 88.0), turned to -90 degrees
- moved C12 88.1 mm to (44.3, 80.0), turned to 90 degrees
- moved C10 86.5 mm to (48.3, 89.0), turned to 180 degrees
- moved C11 86.2 mm to (46.8, 82.8), turned to -90 degrees
- moved C8 85.8 mm to (44.6, 88.0), turned to -90 degrees
- moved FB1 73.0 mm to (48.3, 87.5)
- moved C3 67.7 mm to (63.6, 96.5)
- moved D1 67.2 mm to (63.3, 94.0), turned to 180 degrees
- moved R2 67.1 mm to (51.5, 75.8)
- moved R4 63.9 mm to (53.7, 89.7), turned to 180 degrees
- moved J4 62.1 mm to (50.7, 92.5), turned to 90 degrees
- moved R5 62.0 mm to (55.7, 89.7)
- moved R3 58.4 mm to (59.8, 80.2), turned to -90 degrees
- moved SW1 53.3 mm to (43.6, 72.2)
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Connections:
- J2 pad 1: +3V3 -> +3.3V
- J4 pad 1: +3V3 -> +3.3V
- R4 pad 2: +3V3 -> +3.3V
- R5 pad 2: +3V3 -> +3.3V
Routing:
- net /USB_D-: track 0.00 -> 17.2 mm
- net /USB_D+: track 0.00 -> 17.2 mm
- net /HSE_OUT: track 0.00 -> 9.39 mm
- net /HSE_IN: track 0.00 -> 7.63 mm
- net /USART1_TX: track 0.00 -> 7.39 mm
- net /I2C2_SCL: track 0.00 -> 7.25 mm
- net /USART1_RX: track 0.00 -> 6.91 mm
- net /I2C2_SDA: track 0.00 -> 6.65 mm
- net Net-(C10-Pad2): track 0.00 -> 3.47 mm
- net Net-(U2-BOOT0): track 0.00 -> 2.24 mm
- net /NRST: track 0.00 -> 2.18 mm
- net Net-(C10-Pad1): track 0.00 -> 1.73 mm
- added copper zone on F.Cu, net +3.3V

Commit message: stm32f103 for learn Kicad
Parts:
- moved C12 81.8 mm to (124.8, 94.1)
- moved C13 81.8 mm to (123.3, 99.8)
- moved C2 81.8 mm to (144.1, 105.7)
- moved C4 81.8 mm to (126.8, 93.3)
- moved C6 81.8 mm to (140.9, 91.8)
- moved C9 81.8 mm to (126.6, 102.0)
- moved J2 81.8 mm to (137.8, 85.3)
- moved J3 81.8 mm to (143.5, 85.3)
- moved J4 81.8 mm to (131.3, 106.5)
- moved R1 81.8 mm to (146.7, 107.7)
- moved R2 81.8 mm to (132.0, 89.8)
- moved SW1 81.8 mm to (124.2, 86.3)
- moved Y1 81.8 mm to (122.4, 96.7)
- moved C1 81.8 mm to (152.0, 98.8)
- moved C10 81.8 mm to (128.8, 103.1)
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Routing:
- net +3.3V: track 0.00 -> 113.5 mm, vias 0 -> 2
- net /SWDIO: track 0.00 -> 29.2 mm, vias 0 -> 1
- net /SWCLK: track 0.00 -> 15.8 mm, vias 0 -> 1
- net /SW_BOOTO: track 0.00 -> 12.8 mm
- net VBUS: track 0.00 -> 3.81 mm
- net Net-(D1-K): track 0.00 -> 2.01 mm
- added copper zone on B.Cu, net +3.3V
- added copper zone on B.Cu, net GND
- added copper zone on F.Cu, net GND
- added copper zone on F.Cu, net VBUS
Other:
- board outline added: 51.1 x 34.4 mm
